Commit message: Improve dashboard UI

File: urdf/volvo_ec240cl.urdf (robot description, URDF)
Before this commit: robot gustav, 6 links, 5 joints
Joints:
- joint arm_joint: limit lower=0.698 upper=2.1 effort=1000.0 velocity=0.5 -> lower=0.685 upper=2.751 effort=1000.0 velocity=0.5

Commit message: Set the attachment limits

File: urdf/volvo_ec240cl.urdf (robot description, URDF)
Before this commit: robot gustav, 6 links, 5 joints
Joints:
- joint attachment_joint: limit (none) -> lower=0 upper=3.10 effort=1000.0 velocity=0.5

Commit message: Allow more freedom on the attachment joint

File: urdf/volvo_ec240cl.urdf (robot description, URDF)
Before this commit: robot gustav, 6 links, 5 joints
Joints:
- joint attachment_joint: limit lower=0 upper=3.10 effort=1000.0 velocity=0.5 -> lower=0 upper=3.316 effort=1000.0 velocity=0.5

Commit message: Expand arm joint

File: urdf/volvo_ec240cl.urdf (robot description, URDF)
Before this commit: robot gustav, 6 links, 5 joints
Joints:
- joint arm_joint: limit lower=0.685 upper=2.751 effort=1000.0 velocity=0.5 -> lower=0.685 upper=2.76 effort=1000.0 velocity=0.5

Commit message: Add a fixed end joint to demonstrate the effector

File: urdf/volvo_ec240cl.urdf (robot description, URDF)
Before this commit: robot gustav, 6 links, 5 joints
Joints:
- joint attachment_joint: origin xyz=2.97 0 0 -> xyz=2.97 0 0 rpy=0 -1.5 0

Commit message: Update metrics

File: urdf/volvo_ec240cl.urdf (robot description, URDF)
Before this commit: robot gustav, 6 links, 5 joints
Joints:
- joint boom_joint: origin xyz=0.16 0 0 rpy=0 0 0 -> xyz=0.16 0 0.595 rpy=0 0 0
- joint frame_joint: origin xyz=0 0 1.085 rpy=0 0 0 -> xyz=0 0 1.295 rpy=0 0 0

Commit message: URDF model cleanup

File: urdf/volvo_ec240cl.urdf (robot description, URDF)
Before this commit: robot gustav, 6 links, 5 joints
Joints:
- joint boom_joint: origin xyz=0.16 0 0.595 rpy=0 0 0 -> xyz=0.16 0 0.595
- joint frame_joint: origin xyz=0 0 1.295 rpy=0 0 0 -> xyz=0 0 1.295
- joint undercarriage_joint: origin xyz=0 0 0 rpy=0 0 0 -> (none)

Commit message: Adjust upper and lower bounds on attachment_joint

File: urdf/volvo_ec240cl.urdf (robot description, URDF)
Before this commit: robot gustav, 6 links, 5 joints
Joints:
- joint attachment_joint: limit lower=0 upper=3.316 effort=1000.0 velocity=0.5 -> lower=-0.962 upper=2.138 effort=1000.0 velocity=0.5; origin xyz=2.97 0 0 rpy=0 -1.5 0 -> xyz=2.97 0 0

Commit message: Adjust encoder range

File: urdf/volvo_ec240cl.urdf (robot description, URDF)
Before this commit: robot gustav, 6 links, 5 joints
Joints:
- joint arm_joint: limit lower=0.685 upper=2.76 effort=1000.0 velocity=0.5 -> lower=0.68 upper=2.76 effort=1000.0 velocity=0.5
- joint attachment_joint: limit lower=-0.962 upper=2.138 effort=1000.0 velocity=0.5 -> lower=-0.962 upper=2.19 effort=1000.0 velocity=0.5

Commit message: Show the end joint by default

File: urdf/volvo_ec240cl.urdf (robot description, URDF)
Before this commit: robot gustav, 6 links, 5 joints
Joints:
- added joint end_joint: type fixed, parent arm, child attachment, origin xyz=1.5 0 0, axis 0 1 0

Commit message: continuous joint does not have limits

File: urdf/volvo_ec240cl.urdf (robot description, URDF)
Before this commit: robot gustav, 6 links, 6 joints
Joints:
- joint frame_joint: limit lower=0 upper=6.283 velocity=0.5 -> (none)

Commit message: Set frame to continuous joint

File: urdf/volvo_ec240cl.urdf (robot description, URDF)
Before this commit: robot gustav, 6 links, 6 joints
Joints:
- joint frame_joint: type revolute -> continuous
